File: Mixed_Signal_Board-TNA/mcu.kicad_sch (KiCad schematic)
At the start: 40 parts, among them J200 USB_C_Receptacle_USB2.0_14P, J201 2x5 1.27mm, U200 STM32F103CBT6, U201 USBLC6-2SC6, Y200 16MHz

Commit message: Just Before Layout
Parts:
- FL200: footprint Inductor_THT:L_CommonMode_PulseElectronics_PH9455x105NL_1 -> CMF3216F-900-2P-T:CMF3216F-900-2P-T
Changed lines of the file:
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@@
 					(size 1.27 1.27)
 				)
-				(hide yes)
 			)
 		)
@@
 			)
 		)
-		(property "Footprint" "Inductor_THT:L_CommonMode_PulseElectronics_PH9455x105NL_1"
+		(property "Footprint" "CMF3216F-900-2P-T:CMF3216F-900-2P-T"
 			(at 232.41 144.78 0)
 			(effects
