File: Mixed_Signal_Board-TNA/Mixed_Signal_Board-TNA.kicad_sch (KiCad schematic)
At the start: 0 parts

Commit message: Done Layout
Parts:
- added H1, H2, H3, H4: MountingHole, MountingHole:MountingHole_3.2mm_M3, symbol Mechanical:MountingHole
Other:
- note added: "Mounting Holes (M3)"
