File: Mixed_Signal_Board-TNA/dac.kicad_sch (KiCad schematic)
At the start: 17 parts, among them J400 031-5640-1010, U304 MCP6001T-E/OT, U400 DAC7563SDGSR

Commit message: Just Before Layout
Changed lines of the file:
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@@
 				)
 				(justify left top)
-				(hide yes)
 			)
 		)

Commit message: Done Layout
Other:
- moved on the sheet: R404
Changed lines of the file:
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@@
 	(wire
 		(pts
-			(xy 110.49 82.55) (xy 113.03 82.55)
+			(xy 110.49 82.55) (xy 111.76 82.55)
 		)
 		(stroke
@@
 	(wire
 		(pts
-			(xy 120.65 82.55) (xy 121.92 82.55)
+			(xy 119.38 82.55) (xy 121.92 82.55)
 		)
 		(stroke
@@
 	(symbol
 		(lib_id "Device:R_US")
-		(at 116.84 82.55 270)
+		(at 115.57 82.55 270)
 		(unit 1)
 		(exclude_from_sim no)
@@
 		(dnp no)
 		(property "Reference" "R404"
-			(at 116.84 77.978 90)
+			(at 115.57 77.978 90)
 			(effects
 				(font
@@
 		)
 		(property "Value" "12k"
-			(at 116.84 80.264 90)
+			(at 115.57 80.264 90)
 			(effects
 				(font
@@
 		)
 		(property "Footprint" "Resistor_SMD:R_0402_1005Metric"
-			(at 116.586 83.566 90)
+			(at 115.316 83.566 90)
 			(effects
 				(font
@@
 		)
 		(property "Datasheet" "~"
-			(at 116.84 82.55 0)
+			(at 115.57 82.55 0)
 			(effects
 				(font
@@
 		)
 		(property "Description" "Resistor, US symbol"
-			(at 116.84 82.55 0)
-			(effects
-				(font
+			(at 115.57 82.55 0)
+			(effects
+				(font
