File: Mixed_Signal_Board-TNA/power.kicad_sch (KiCad schematic)
At the start: 22 parts, among them U100 HT7533, U102 TLV62569DBV, U2 MCP6001T-E/OT

Commit message: Just Before Layout
Other:
- note added: "- 0.5mm for Power - 0.3mm for Signal - Spacing 3 x Dielectric Thickness - Always Minimize Length - Maximise Spacing"
- note added: "- Signals flow in closed loops - Signal energy travels in dielectric material - Signals in kHz range, return current will be directly underneath the forward current trace - Better with low impedance return path - Stitching Vias"
- note added: "- Small 0.45mm pad, 0.25mm drill - Medium 0.7mm pad, 0.3mm drill (Usually) - Large 0.8mm pad, 0.4mm drill"
- note added: "- Trace Length vs Rise Time - l_trace >= (t_r/2)*v_propagation - where t_r = 10-90% rise/fall time - v_propagation ~6in/ns in FR4 - minimise reflections - Trace Impedance, Z_o=sqrt(L/C)"
- note added: "Controlled Impedances:"
- note added: "PCB Facts:"
- note added: "Rules of Thumb:"
- note added: "Via Recommendation"
Changed lines of the file:
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@@
+		)
+	)
+	(text "Rules of Thumb:\n"
+		(exclude_from_sim no)
+		(at 216.154 105.41 0)
+		(effects
+			(font
+				(size 1.27 1.27)
+				(thickness 0.254)
+				(bold yes)
+			)
 		)
 	)
@@
 				(size 1.27 1.27)
 			)
+		)
+	)
+	(text "- Small  0.45mm pad, 0.25mm drill\n- Medium 0.7mm pad, 0.3mm drill (Usually)\n- Large  0.8mm pad, 0.4mm drill"
+		(exclude_from_sim no)
+		(at 209.804 143.256 0)
+		(effects
+			(font
+				(size 1.27 1.27)
+			)
+			(justify left)
 		)
 	)
@@
 				(bold yes)
 			)
+		)
+	)
+	(text "- Signals flow in closed loops\n- Signal energy travels in dielectric material\n- Signals in kHz range, return current will be \n  directly underneath the forward current trace\n- Better with low impedance return path\n- Stitching Vias"
+		(exclude_from_sim no)
+		(at 207.772 96.266 0)
+		(effects
+			(font
+				(size 1.27 1.27)
+			)
+			(justify left)
 		)
 	)
@@
 		)
 	)
-	(text "Recommended:\n- 0402, 0603, 0805 onwards\n- SOT Packages"
-		(exclude_from_sim no)
-		(at 169.418 41.148 0)
-		(effects
-			(font
-				(size 1.27 1.27)
-				(thickness 0.1588)
-			)
-			(justify left)
-		)
-	)
-	(text "100mA max"
-		(exclude_from_sim no)
-		(at 98.044 64.516 0)
-		(effects
-			(font
-				(size 1.27 1.27)
-			)
-			(justify left)
-		)
-	)
-	(text "Pi Filter Network"
-		(exclude_from_sim no)
-		(at 33.782 76.708 0)
+	(text "Via Recommendation"
+		(exclude_from_sim no)
+		(at 209.296 137.922 0)
 		(effects
 			(font
@@
 				(bold yes)
 			)
-		)
-	)
-	(text "Current Limiting Resistor"
-		(exclude_from_sim no)
-		(at 172.212 118.364 0)
+			(justify left)
+		)
+	)
+	(text "Recommended:\n- 0402, 0603, 0805 onwards\n- SOT Packages"
+		(exclude_from_sim no)
+		(at 169.418 41.148 0)
+		(effects
+			(font
+				(size 1.27 1.27)
+				(thickness 0.1588)
+			)
+			(justify left)
+		)
+	)
+	(text " - Trace Length vs Rise Time\n - l_trace >= (t_r/2)*v_propagation\n - where t_r = 10-90% rise/fall time\n - v_propagation ~6in/ns in FR4 \n - minimise reflections\n - Trace Impedance, Z_o=sqrt(L/C)"
+		(exclude_from_sim no)
+		(at 207.264 128.27 0)
+		(effects
+			(font
+				(size 1.27 1.27)
+			)
+			(justify left)
+		)
+	)
+	(text "100mA max"
+		(exclude_from_sim no)
+		(at 98.044 64.516 0)
+		(effects
+			(font
+				(size 1.27 1.27)
+			)
+			(justify left)
+		)
+	)
+	(text "Pi Filter Network"
+		(exclude_from_sim no)
+		(at 33.782 76.708 0)
 		(effects
 			(font
@@
 		)
 	)
-	(text "Buck Converter"
-		(exclude_from_sim no)
-		(at 94.488 131.064 0)
+	(text "Current Limiting Resistor"
+		(exclude_from_sim no)
+		(at 172.212 118.364 0)
 		(effects
 			(font
@@
 		)
 	)
-	(text "Voltage Follower"
-		(exclude_from_sim no)
-		(at 254.254 42.926 0)
+	(text "Buck Converter"
+		(exclude_from_sim no)
+		(at 94.488 131.064 0)
 		(effects
 			(font
@@
 		)
 	)
-	(text "Low Pass RC Filter"
-		(exclude_from_sim no)
-		(at 73.66 42.418 0)
+	(text "Voltage Follower"
+		(exclude_from_sim no)
+		(at 254.254 42.926 0)
 		(effects
 			(font
@@
 		)
 	)
+	(text "Low Pass RC Filter"
+		(exclude_from_sim no)
+		(at 73.66 42.418 0)
+		(effects
+			(font
+				(size 1.27 1.27)
+				(thickness 0.254)
+				(bold yes)
+			)
+		)
+	)
 	(text "L=[V_out*(V_in-V_out)]/(V_in*f_sw*delta_IL)\nwhere delta_IL = k*IL\nL=[3.3*(5-3.3)]/(5*1.5MHz*(0.25^0.25A)) = 12uH\nStandard Value = 15uH\nLighter Loads -> Larger Inductors"
 		(exclude_from_sim no)
@@
 		(exclude_from_sim no)
 		(at 25.908 81.28 0)
+		(effects
+			(font
+				(size 1.27 1.27)
+			)
+			(justify left)
+		)
+	)
+	(text "- 0.5mm for Power\n- 0.3mm for Signal\n- Spacing 3 x Dielectric Thickness\n- Always Minimize Length\n- Maximise Spacing"
+		(exclude_from_sim no)
+		(at 208.026 112.014 0)
 		(effects
 			(font
@@
 		)
 	)
+	(text "PCB Facts:\n"
+		(exclude_from_sim no)
+		(at 213.106 88.646 0)
+		(effects
+			(font
+				(size 1.27 1.27)
+				(thickness 0.254)
+				(bold yes)
+			)
+		)
+	)
 	(text "DCR=0R15\n"
 		(exclude_from_sim no)
@@
 			)
 			(justify left)
+		)
+	)
+	(text "Controlled Impedances:"
+		(exclude_from_sim no)
+		(at 219.964 120.65 0)
+		(effects
+			(font
+				(size 1.27 1.27)
+				(thickness 0.254)
+				(bold yes)
+			)
 		)
 	)
@@
 					(size 1.27 1.27)
 				)
-				(hide yes)
 			)
 		)
@@
 					(size 1.27 1.27)
 				)
-				(hide yes)
 			)
 		)
@@
 					(size 1.27 1.27)
 				)
-				(hide yes)
-			)
-		)
+			)
+		)

Commit message: Done Layout
Parts:
- C106: footprint (none) -> Capacitor_SMD:C_0402_1005Metric
Changed lines of the file:
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@@
 		(fields_autoplaced yes)
 		(property "Reference" "U102"
-			(at 95.25 99.06 0)
+			(at 95.25 97.79 0)
 			(effects
 				(font
@@
 		)
 		(property "Value" "TLV62569DBV"
-			(at 95.25 101.6 0)
+			(at 95.25 100.33 0)
 			(effects
 				(font
@@
 					(size 1.27 1.27)
 				)
+				(hide yes)
 			)
 		)
@@
 					(size 1.27 1.27)
 				)
+				(hide yes)
 			)
 		)
@@
 			)
 		)
-		(property "Footprint" ""
+		(property "Footprint" "Capacitor_SMD:C_0402_1005Metric"
 			(at 158.4452 114.3 0)
 			(effects
@@
 		(dnp no)
 		(property "Reference" "U2"
-			(at 252.73 54.5398 0)
+			(at 246.888 55.626 0)
 			(effects
 				(font
@@
 		)
 		(property "Footprint" "MCP6001T-E_OT:SOT95P270X145-5N"
-			(at 245.11 59.69 0)
-			(effects
-				(font
-					(size 1.27 1.27)
-				)
-			)
-		)
+			(at 254.254 68.834 0)
+			(effects
+				(font
+					(size 1.27 1.27)
+				)
+				(hide yes)
+			)
+		)
